File: cacophony-blocks.kicad_blocks/5V-buck-boost.kicad_block/5V-buck-boost.kicad_sch (KiCad schematic)
At the start: 16 parts, among them U201 TPS63070

Commit message: Update 5V buck-boost design block
Parts:
- added R5: 10k, Resistor_SMD:R_0402_1005Metric, symbol Device:R
- renumbered R219 to R1, R216 to R2, R218 to R3
Connections:
- net BUCK_BOOST_FPWM is gone; now on net 5V_EN: U201.1 (PS/SYNC)
- net 5V_EN: now also R5.2
- net +5V: now reaches FB1.2
- net VCC: no longer names the net of C203.1, C203.1, C204.1, U201.12,13 (Vin)
- net VCC: now also R5.1
Other:
- moved on the sheet: C203, C204, C205, C206, C207, C208, C209, C210, FB1, L3, R1, R2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
