File: cacophony-blocks.kicad_blocks/5V-buck-boost.kicad_block/5V-buck-boost.kicad_pcb (KiCad board)
At the start: 4 copper layers, 17 parts, among them U1 TPS63070

Commit message: Update library for solar-tester
Routing:
- net GND: track 6.58 -> 6.44 mm, vias 32 -> 30
