File: cacophony-blocks/5V-buck-boost/5V-buck-boost.kicad_sch (KiCad schematic)
At the start: 17 parts, among them U1 TPS63070

Commit message: Update 5V buck-boost design block
Other:
- moved on the sheet: C1, C2, C3, C4, C5, C6, C7, C8, C9, FB1, L1, R1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
